File: projects/rc_vehicle/stm32_espc3_schemas/stm32_car_telemetry.kicad_pcb (KiCad board)
At the start: 2 copper layers, 43 parts, among them SW1 CK_KMS2xxG, U1 STM32G431CBTxZ, U2 LP5907MFX-3.3, U3 LSM6DSM, U4 TXS0104ED, U5 ESP32-C3-DevKitM-1, Y1 16MHz, Y2 32.768 kHz

Commit message: update stm32g4 pcb
Parts:
- removed 5V1: Conn_01x02_Pin, Connector_PinHeader_2.54mm:PinHeader_1x02_P2.54mm_Vertical
- removed C6: 100nF, Capacitor_SMD:C_0201_0603Metric
- removed ESP_IO1: Conn_01x11_Pin, Connector_PinHeader_2.54mm:PinHeader_1x11_P2.54mm_Vertical
- removed ESP_IO1: Conn_01x13_Pin, Connector_PinSocket_2.54mm:PinSocket_1x13_P2.54mm_Vertical
- removed R1: 0, Resistor_SMD:R_0201_0603Metric
- removed R2: NI, Resistor_SMD:R_0201_0603Metric
- removed STM_GPIO1, STM_GPIO2: Conn_01x12_Pin, Connector_PinHeader_2.54mm:PinHeader_1x12_P2.54mm_Vertical
- removed SW1: CK_KMS2xxG, Button_Switch_SMD:SW_SPST_CK_KMS2xxGP
- C12, C13, C17, C18: footprint Capacitor_SMD:C_0805_2012Metric -> Capacitor_SMD:C_01005_0402Metric
- NRST_Button1: footprint Button_Switch_SMD:SW_SPST_PTS647_Sx38 -> Button_Switch_SMD:SW_SPST_PTS810
- moved C14 96.0 mm to (126.2, 51.0), turned to -90 degrees
- moved C15 91.4 mm to (135.1, 50.5), turned to 90 degrees
- moved U4 90.9 mm to (127.0, 87.5), turned to -90 degrees
- moved C16 89.9 mm to (140.0, 50.5), turned to 90 degrees
- moved Y2 86.8 mm to (126.2, 65.6), turned to 90 degrees
- moved R3 85.5 mm to (133.0, 62.9), turned to 90 degrees
- moved Y1 83.6 mm to (124.2, 70.8), turned to 90 degrees
- moved R4 76.2 mm to (144.4, 67.5), turned to 180 degrees
- moved C11 65.0 mm to (123.7, 75.3), turned to 180 degrees
- moved SWD1 64.5 mm to (118.2, 61.7)
- moved U5 63.5 mm to (151.5, 47.9), turned to 0 degrees
- moved Servo_Signal1 62.6 mm to (142.0, 90.8), turned to 180 degrees
- moved U1 58.0 mm to (134.3, 69.2)
- moved NRST_Button1 56.3 mm to (123.7, 79.4), turned to 90 degrees
- moved C18 54.7 mm to (129.2, 64.0), turned to 90 degrees
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Connections:
- C10 pad 2: /VREF -> /3V3
- C12 pad 1: /OSC_IN -> /OSC_OUT
- C13 pad 1: /OSC_OUT -> /OSC_IN
- C17 pad 1: /OSC32_IN -> /OSC32_OUT
- C18 pad 1: /OSC32_OUT -> /OSC32_IN
- U1 pad 10: /UART_TX_STM -> /STEERING_OUT
- U1 pad 11: /UART_RX_STM -> /THROTTLE_OUT
- U1 pad 12: /PA4 -> unconnected-(U1-PA4-Pad12)
- U1 pad 13: /PA5 -> unconnected-(U1-PA5-Pad13)
- U1 pad 14: /PA6 -> unconnected-(U1-PA6-Pad14)
- U1 pad 15: /PA7 -> unconnected-(U1-PA7-Pad15)
- U1 pad 16: /PB0 -> unconnected-(U1-PB0-Pad16)
- U1 pad 17: /PB1 -> unconnected-(U1-PB1-Pad17)
- U1 pad 18: /PB2 -> unconnected-(U1-PB2-Pad18)
- U1 pad 2: /PC13 -> unconnected-(U1-PC13-Pad2)
- U1 pad 20: /VREF -> /3V3
- U1 pad 22: /PB10 -> unconnected-(U1-PB10-Pad22)
- U1 pad 25: /PB11 -> unconnected-(U1-PB11-Pad25)
- U1 pad 30: /THROTTLE_OUT -> /ESP_RST
- U1 pad 31: /STEERING_OUT -> /UART_TX_STM
- U1 pad 32: /PA10 -> /UART_RX_STM
- U1 pad 33: /PA11 -> unconnected-(U1-PA11-Pad33)
- U1 pad 34: /PA12 -> unconnected-(U1-PA12-Pad34)
- U1 pad 39: /ESP_RST -> unconnected-(U1-PA15-Pad39)
- U1 pad 40: /PB3 -> unconnected-(U1-PB3-Pad40)
- U1 pad 41: /PB4 -> unconnected-(U1-PB4-Pad41)
- U1 pad 42: /PB5 -> unconnected-(U1-PB5-Pad42)
- U1 pad 43: /PB6 -> unconnected-(U1-PB6-Pad43)
- U1 pad 44: /PB7 -> unconnected-(U1-PB7-Pad44)
- U1 pad 46: /PB9 -> unconnected-(U1-PB9-Pad46)
- U1 pad 8: /THROTTLE_IN_PWM -> /STEERING_IN_PWM
- U1 pad 9: /STEERING_IN_PWM -> /THROTTLE_IN_PWM
- U5 pad 10: /ESP_IO1 -> unconnected-(U5-IO1-Pad10)
- U5 pad 11: /ESP_IO10 -> unconnected-(U5-IO10-Pad11)
- U5 pad 17: /ESP_IO19 -> unconnected-(U5-IO19-Pad17)
- U5 pad 18: /ESP_IO18 -> unconnected-(U5-IO18-Pad18)
- U5 pad 20: /ESP_IO4 -> unconnected-(U5-IO4-Pad20)
- U5 pad 21: /ESP_IO5 -> unconnected-(U5-IO5-Pad21)
- U5 pad 22: /ESP_IO6 -> unconnected-(U5-IO6-Pad22)
- U5 pad 23: /ESP_IO7 -> unconnected-(U5-IO7-Pad23)
- U5 pad 25: /ESP_IO8 -> unconnected-(U5-IO8-Pad25)
- U5 pad 26: /ESP_IO9 -> unconnected-(U5-IO9-Pad26)
- U5 pad 4: /ESP_IO2 -> unconnected-(U5-IO2-Pad4)
- U5 pad 5: /ESP_IO3 -> unconnected-(U5-IO3-Pad5)
- U5 pad 9: /ESP_IO0 -> unconnected-(U5-IO0-Pad9)
- Y1 pad 1: /OSC_IN -> /OSC_OUT
- Y1 pad 2: /OSC_OUT -> /OSC_IN
- Y2 pad 1: /OSC32_IN -> /OSC32_OUT
- Y2 pad 2: /OSC32_OUT -> /OSC32_IN
Routing:
- net /3V3: track 0.00 -> 276.4 mm, vias 0 -> 4
- net /5V: track 0.00 -> 152.8 mm, vias 0 -> 1
- net GND: track 11.6 -> 71.8 mm, vias 0 -> 7
- net /UART_RX_STM: track 0.00 -> 43.3 mm
- net /UART_TX_STM: track 0.00 -> 42.5 mm
- net /NRST: track 0.00 -> 33.2 mm
- net Net-(RC_Receiver_CH2-Pin_2): track 0.00 -> 30.0 mm
- net /SWCLK: track 0.00 -> 26.1 mm
- net /SWDIO: track 0.00 -> 24.6 mm
- net Net-(RC_Receiver_CH1-Pin_2): track 0.00 -> 23.3 mm
- net /STEERING_IN_PWM: track 0.00 -> 18.2 mm
- net /THROTTLE_IN_PWM: track 0.00 -> 17.2 mm
- net Net-(Servo_Signal1-Pin_2): track 0.00 -> 16.6 mm
- net /STEERING_OUT: track 0.00 -> 16.2 mm
- net /THROTTLE_OUT: track 0.00 -> 15.7 mm
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- added copper zone on F.Cu, net (none)
- added copper zone on B.Cu, net GND
- added copper zone on F.Cu, net GND
Other:
- board outline added: 64 x 50.5 mm
