File: projects/rc_vehicle/stm32_espc3_schemas/stm32_car_telemetry.kicad_sch (KiCad schematic)
At the start: 39 parts, among them U1 STM32G431CBTxZ, U2 LP5907MFX-3.3, U3 LSM6DSM, U4 TXS0104ED, U5 ESP32-C3-DevKitM-1, Y1 16MHz, Y2 32.768 kHz

Commit message: update stm32g4 pcb
Parts:
- removed ESP_IO1: Conn_01x13_Pin, Connector_PinSocket_2.54mm:PinSocket_1x13_P2.54mm_Vertical, symbol Connector:Conn_01x13_Pin
- removed R1: 0, Resistor_SMD:R_0201_0603Metric, symbol Device:R
- removed R2: NI, Resistor_SMD:R_0201_0603Metric, symbol Device:R
- removed STM_GPIO1, STM_GPIO2: Conn_01x12_Pin, Connector_PinHeader_2.54mm:PinHeader_1x12_P2.54mm_Vertical, symbol Connector:Conn_01x12_Pin
- C12, C13, C17, C18: footprint Capacitor_SMD:C_0805_2012Metric -> Capacitor_SMD:C_01005_0402Metric
- NRST_Button1: footprint Button_Switch_SMD:SW_SPST_PTS647_Sx38 -> Button_Switch_SMD:SW_SPST_PTS810
Connections:
- net PA10 is gone; now on net UART_RX_STM: U1.32 (PA10)
- net VREF is gone; now on net 3V3: C10.2, U1.20 (VREF+)
- net ESP_RST: now also U1.30 (PA8); no longer U1.39 (PA15)
- net OSC32_IN: now also C18.1, Y2.2; no longer C17.1, Y2.1
- net OSC32_OUT: now also C17.1, Y2.1; no longer C18.1, Y2.2
- net OSC_IN: now also C13.1, Y1.2; no longer C12.1, Y1.1
- net OSC_OUT: now also C12.1, Y1.1; no longer C13.1, Y1.2
- net STEERING_IN_PWM: now also U1.8 (PA0); no longer U1.9 (PA1)
- net STEERING_OUT: now also U1.10 (PA2); no longer U1.31 (PA9)
- net THROTTLE_IN_PWM: now also U1.9 (PA1); no longer U1.8 (PA0)
- net THROTTLE_OUT: now also U1.11 (PA3); no longer U1.30 (PA8)
- net UART_RX_STM: no longer U1.11 (PA3)
- net UART_TX_STM: now also U1.31 (PA9); no longer U1.10 (PA2)
- net ESP_IO0: no longer names the net of U5.9 (IO0)
- net ESP_IO1: no longer names the net of U5.10 (IO1)
- net ESP_IO10: no longer names the net of U5.11 (IO10)
- net ESP_IO18: no longer names the net of U5.18 (IO18)
- net ESP_IO19: no longer names the net of U5.17 (IO19)
- net ESP_IO2: no longer names the net of U5.4 (IO2)
- net ESP_IO3: no longer names the net of U5.5 (IO3)
- net ESP_IO4: no longer names the net of U5.20 (IO4)
- net ESP_IO5: no longer names the net of U5.21 (IO5)
- net ESP_IO6: no longer names the net of U5.22 (IO6)
- net ESP_IO7: no longer names the net of U5.23 (IO7)
- net ESP_IO8: no longer names the net of U5.25 (IO8)
- net ESP_IO9: no longer names the net of U5.26 (IO9)
- net PA11: no longer names the net of U1.33 (PA11)
- net PA12: no longer names the net of U1.34 (PA12)
- net PA4: no longer names the net of U1.12 (PA4)
- net PA5: no longer names the net of U1.13 (PA5)
- net PA6: no longer names the net of U1.14 (PA6)
- net PA7: no longer names the net of U1.15 (PA7)
- net PB0: no longer names the net of U1.16 (PB0)
- net PB1: no longer names the net of U1.17 (PB1)
- net PB10: no longer names the net of U1.22 (PB10)
- net PB11: no longer names the net of U1.25 (PB11)
- net PB2: no longer names the net of U1.18 (PB2)
- net PB3: no longer names the net of U1.40 (PB3)
- net PB4: no longer names the net of U1.41 (PB4)
- net PB5: no longer names the net of U1.42 (PB5)
- net PB6: no longer names the net of U1.43 (PB6)
- net PB7: no longer names the net of U1.44 (PB7)
- net PB9: no longer names the net of U1.46 (PB9)
- net PC13: no longer names the net of U1.2 (PC13)
- no-connect marks 7 -> 39
